File: hardware/keys.kicad_sch (KiCad schematic)
At the start: 41 parts, among them SW10 SW_Push, SW11 SW_Push, SW12 SW_Push, SW4 SW_Push, SW5 SW_Push, SW6 SW_Push, SW7 SW_Push, SW8 SW_Push, SW9 SW_Push

Commit message: Updated artwork Added as-built rev 1 PCB
Connections:
- net +3.3V: now also JP1.3 (B); no longer JP1.1 (A)
- net VCC: now also JP1.1 (A); no longer JP1.3 (B)
Other:
- moved on the sheet: C15, C16, C17, C18, C19, C20, D10, D11, D12, D13, D14, D15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
