File: hardware/mk9-badge.kicad_pcb (KiCad board)
At the start: 2 copper layers, 75 x 75 mm, 92 parts, among them J1 USB-C, SW1 Boot Select, SW10 SW_Push, SW11 SW_Push, SW12 SW_Push, SW2 SW_SPDT, SW3 Reset, SW4 SW_Push, SW5 SW_Push, SW6 SW_Push, SW7 SW_Push, SW8 SW_Push, SW9 SW_Push, U1 GSDA213, U2 RP2040, U3 NCP115ASN330T2G, U4 W25Q128JVSIM, X1 Badgelife_sao_connector_v169b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, X2 Badgelife_sao_connector_v169b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, Y1 ABM8-272-T3

Commit message: Updated artwork Added as-built rev 1 PCB
Parts:
- moved TP6 3.79 mm to (111.0, 66.4)
- moved TP5 3.18 mm to (111.0, 62.0)
- moved G*** 2.71 mm to (108.4, 77.8)
- moved J1 1.78 mm to (138.2, 42.6)
- moved C3 1.62 mm to (111.5, 70.2)
- moved U1 1.53 mm to (114.6, 70.9)
- moved G*** 0.26 mm to (138.3, 77.7)
- moved R3 0.21 mm to (144.8, 47.7)
- turned JP1 to 0 degrees
Connections:
- JP1 pad 1: +3.3V -> VCC
- JP1 pad 3: VCC -> +3.3V
Routing:
- net GND: track 107.3 -> 122.9 mm, vias 37 -> 38
- net Net-(D22-DOUT): track 24.1 -> 32.8 mm
- net +3.3V: track 213.0 -> 217.9 mm, vias 6 -> 7
- net VBUS: track 15.5 -> 19.1 mm
- net Net-(D1-K-Pad2): track 15.6 -> 19.2 mm
- net Net-(D1-K-Pad1): track 18.0 -> 19.4 mm
- net Net-(J1-CC1): track 6.79 -> 7.86 mm
- net Net-(J1-CC2): track 6.51 -> 7.50 mm
- net SDA1: track 11.4 -> 12.3 mm
- net SCL1: track 10.5 -> 11.3 mm
- net VCC: vias 2 -> 3
Other:
- board text added: "@hamster"
- board text added: "BOOT"
- board text added: "RESET"
